File: 01-ALU_Trilogy/01.2 - Breadboard/Revised_Schematic/Revised_Schematic.kicad_sch (KiCad schematic)
At the start: 13 parts, among them SW1 A(4), SW2 B(4), SW3 s(3), U1 74HC04, U2 74HC04

Commit message: Improve README
Parts:
- removed R5, R6, R7, R8: 10k, symbol Device:R_US
- added C1, C10, C11, C12, C13, C14, C15, C2, C3, C4, C5, C6, C7, C8, C9: 0.1μF, symbol Device:C
- added D1, D2, D3, D4: LED, symbol Device:LED
- added R41, R42, R43, R44, R45, R46, R47, R48, R49, R50, R51: 10k, symbol Device:R_US
- added U10, U11, U12, U13, U14, U15, U7, U9: 74LS157, symbol 74xx:74LS157
- added U3: 74HC00, symbol 74xx:74HC00
- added U4: 74HC86, symbol 74xx:74HC86
- added U5: 74HC32, symbol 74xx:74LS32
- added U6: 74HC08, symbol 74xx:74LS08
- added U8: 74LS283, symbol 74xx:74LS283
- R1, R2, R3, R4: value 10k -> 220Ω
Connections:
- net +5V: now also C1.2, C10.2, C11.2, C12.2, C13.2, C14.2, C15.2, C2.2, C3.2, C4.2, C5.2, C6.2, C7.2, C8.2, C9.2, U10.16 (VCC), U11.16 (VCC), U12.16 (VCC), U13.16 (VCC), U14.16 (VCC), U15.16 (VCC), U3.14 (VCC), U4.14 (VCC), U5.14 (VCC), U6.14 (VCC), U7.16 (VCC), U8.16 (VCC), U9.16 (VCC)
- net at SW1.5, U2.9: now also R47.1, U3.12, U4.12, U5.12, U6.12, U8.12 (A4)
- net at SW1.6, U2.5: now also R48.1, U3.9, U4.9, U5.9, U6.9, U8.14 (A3)
- net at SW1.7, U2.3: now also R46.1, U3.4, U4.4, U5.4, U6.4, U8.3 (A2)
- net at SW1.8, U2.1: now also R45.1, U3.1, U4.1, U5.1, U6.1, U8.5 (A1)
- net at U2.2: now also U10.2 (I0a)
- net at SW2.6, U1.5: now also R43.1, U3.10, U4.10, U5.10, U6.10, U7.10 (I1c); no longer R3.2
- net at U1.6: now also U7.11 (I0c), U9.11 (I0c)
- net at U2.4: now also U10.5 (I0b)
- net at SW2.7, U1.3: now also R42.1, U3.5, U4.5, U5.5, U6.5, U7.6 (I1b); no longer R2.2
- net at U1.4: now also U7.5 (I0b), U9.5 (I0b)
- net at SW2.8, U1.1: now also R41.1, U3.2, U4.2, U5.2, U6.2, U7.3 (I1a); no longer R1.2
- net at U1.2: now also U7.2 (I0a), U9.2 (I0a)
- net GND: now reaches U2.7 (GND)
- net GND: now also U1.7 (GND), C1.1, C10.1, C11.1, C12.1, C13.1, C14.1, C15.1, C2.1, C3.1, C4.1, C5.1, C6.1, C7.1, C8.1, C9.1, D1.1 (K), D2.1 (K), D3.1 (K), D4.1 (K), R41.2, R42.2, R43.2, R44.2, R45.2, R46.2, R47.2, R48.2, R49.2, R50.2, R51.2, U10.15 (E), U10.8 (GND), U11.15 (E), U11.8 (GND), U12.15 (E), U12.8 (GND), U13.15 (E), U13.8 (GND), U14.15 (E), U14.8 (GND), U15.15 (E), U15.8 (GND), U3.7 (GND), U4.7 (GND), U5.7 (GND), U6.7 (GND), U7.15 (E), U7.8 (GND), U8.8 (GND), U9.15 (E), U9.8 (GND)
- net at SW2.5, U1.9: now also R44.1, U3.13, U4.13, U5.13, U6.13, U7.13 (I1d); no longer R4.2
- net at SW3.4: now also R49.1, U15.1 (S), U7.1 (S), U8.7 (C0)
- net at SW3.5: now also R50.1, U13.1 (S), U14.1 (S)
- net at SW3.6: now also R51.1, U10.1 (S), U11.1 (S), U12.1 (S), U9.1 (S)
- net at U2.6: now also U10.11 (I0c)
- net at U1.8: now also U7.14 (I0d), U9.14 (I0d)
- net at U2.8: now also U10.14 (I0d)
- new net: U5.8, U9.10 (I1c)
- new net: U13.14 (I0d), U9.12 (Zd)
- new net: U5.11, U9.13 (I1d)
- new net: U5.3, U9.3 (I1a)
- new net: U13.2 (I0a), U9.4 (Za)
- new net: U5.6, U9.6 (I1b)
- new net: U13.5 (I0b), U9.7 (Zb)
- new net: U13.11 (I0c), U9.9 (Zc)
- new net: U10.3 (I1a), U6.3
- new net: U10.10 (I1c), U6.8
- new net: R2.1, U15.7 (Zb)
- new net: D2.2 (A), R2.2
- new net: U12.11 (I0c), U4.8
- new net: U10.12 (Zd), U13.13 (I1d)
- new net: U10.13 (I1d), U6.11
- new net: U10.4 (Za), U13.3 (I1a)
- new net: U10.6 (I1b), U6.6
- new net: U10.7 (Zb), U13.6 (I1b)
- new net: U10.9 (Zc), U13.10 (I1c)
- new net: U14.9 (Zc), U15.10 (I1c)
- new net: U13.9 (Zc), U15.11 (I0c)
- new net: R4.1, U15.12 (Zd)
- new net: U14.12 (Zd), U15.13 (I1d)
- new net: U13.12 (Zd), U15.14 (I0d)
- new net: U13.4 (Za), U15.2 (I0a)
- new net: U14.4 (Za), U15.3 (I1a)
- new net: R1.1, U15.4 (Za)
- new net: U13.7 (Zb), U15.5 (I0b)
- new net: U14.7 (Zb), U15.6 (I1b)
- new net: R3.1, U15.9 (Zc)
- new net: D1.2 (A), R1.2
- new net: D4.2 (A), R4.2
- new net: D3.2 (A), R3.2
- new net: U11.10 (I1c), U12.10 (I1c), U8.13 (S3)
- new net: U12.12 (Zd), U14.13 (I1d)
- new net: U11.13 (I1d), U12.13 (I1d), U8.10 (S4)
- new net: U12.14 (I0d), U4.11
- new net: U12.2 (I0a), U4.3
- new net: U11.3 (I1a), U12.3 (I1a), U8.4 (S1)
- new net: U12.4 (Za), U14.3 (I1a)
- new net: U12.5 (I0b), U4.6
- new net: U11.6 (I1b), U12.6 (I1b), U8.1 (S2)
- new net: U12.7 (Zb), U14.6 (I1b)
- new net: U12.9 (Zc), U14.10 (I1c)
- new net: U11.2 (I0a), U3.3
- new net: U11.5 (I0b), U3.6
- new net: U11.11 (I0c), U3.8
- new net: U11.12 (Zd), U14.14 (I0d)
- new net: U11.14 (I0d), U3.11
- new net: U11.4 (Za), U14.2 (I0a)
- new net: U11.7 (Zb), U14.5 (I0b)
- new net: U11.9 (Zc), U14.11 (I0c)
- new net: U7.12 (Zd), U8.11 (B4)
- new net: U7.9 (Zc), U8.15 (B3)
- new net: U7.7 (Zb), U8.2 (B2)
- new net: U7.4 (Za), U8.6 (B1)
Other:
- moved on the sheet: SW3, U1A, U1B, U1C, U1D, U1E, U1F, U1G, U2A, U2B, U2C, U2D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
